Commit message: them 2 banh chu dong

File: boe_robot_description/urdf/boe_robot.urdf.xacro (robot description, xacro)
@@ -3,31 +3,83 @@
   xmlns:xacro="http://www.ros.org/wiki/xacro"
   name="boe_robot">
-  <!-- Màu sắc -->
+  <!-- Các thông số chính của robot -->
+  <xacro:property name="wheel_radius" value="0.03272"/>
+  <xacro:property name="wheel_separation" value="0.115"/>
+  <!-- Màu thân xe -->
   <material name="body_color">
     <color rgba="0.796 0.824 0.937 1.0"/>
   </material>
+  <!-- Màu bánh xe -->
+  <material name="wheel_color">
+    <color rgba="0.12 0.12 0.12 1.0"/>
+  </material>
   <!--
-    base_footprint là hình chiếu của tâm robot xuống mặt đất.
-    Link này không có hình dạng và không có khối lượng.
+    base_footprint nằm trên mặt đất,
+    ở gần tâm giữa hai bánh chủ động.
   -->
   <link name="base_footprint"/>
   <!--
-    Đưa base_link lên khỏi mặt đất khoảng 32.2 mm.
-    Giá trị này được tính gần đúng từ bán kính bánh xe.
+    Dịch base_link so với tâm hai bánh:
+    x = -0.03193 m
+    y =  0.004294 m
+    z =  0.03215 m
   -->
   <joint name="base_footprint_joint" type="fixed">
     <parent link="base_footprint"/>
     <child link="base_link"/>
-    <origin xyz="0 0 0.0322" rpy="0 0 0"/>
+    <origin
+      xyz="-0.0319316266 0.0042939669 0.03215"
+      rpy="0 0 0"/>
   </joint>
-  <!-- Khung thân chính của robot -->
+  <!-- Thân xe -->
   <link name="base_link">
     <visual>
       <origin xyz="0 0 0" rpy="0 0 0"/>
       <geometry>
-        <mesh filename="package://boe_robot_description/meshes/base_link.STL"/>
+        <mesh
+          filename="package://boe_robot_description/meshes/base_link.STL"/>
       </geometry>
       <material name="body_color"/>
     </visual>
   </link>
+  <!-- Bánh chủ động bên trái -->
+  <link name="wheel_left_link">
+    <visual>
+      <origin xyz="0 0 0" rpy="0 0 0"/>
+      <geometry>
+        <mesh
+          filename="package://boe_robot_description/meshes/wheel_left_link.STL"/>
+      </geometry>
+      <material name="wheel_color"/>
+    </visual>
+  </link>
+  <joint name="wheel_left_joint" type="continuous">
+    <parent link="base_link"/>
+    <child link="wheel_left_link"/>
+    <origin
+      xyz="0.0329316266 0.0532060331 0.0005737626"
+      rpy="1.5707963268 0 3.1415926536"/>
+    <axis xyz="0 0 1"/>
+    <limit effort="1.0" velocity="20.0"/>
+  </joint>
+  <!-- Bánh chủ động bên phải -->
+  <link name="wheel_right_link">
+    <visual>
+      <origin xyz="0 0 0" rpy="0 0 0"/>
+      <geometry>
+        <mesh
+          filename="package://boe_robot_description/meshes/wheel_right_link.STL"/>
+      </geometry>
+      <material name="wheel_color"/>
+    </visual>
+  </link>
+  <joint name="wheel_right_joint" type="continuous">
+    <parent link="base_link"/>
+    <child link="wheel_right_link"/>
+    <origin
+      xyz="0.0309316266 -0.0617939669 0.0005737626"
+      rpy="1.5707963268 0 0"/>
+    <axis xyz="0 0 -1"/>
+    <limit effort="1.0" velocity="20.0"/>
+  </joint>
 </robot>

Commit message: 1 banh caster

File: boe_robot_description/urdf/boe_robot.urdf.xacro (robot description, xacro)
@@ -83,3 +83,64 @@
     <limit effort="1.0" velocity="20.0"/>
   </joint>
+  <!-- ====================================================== -->
+  <!-- Cụm bánh caster                                       -->
+  <!-- ====================================================== -->
+  <!-- Đế caster được gắn cố định với thân robot -->
+  <link name="caster_base_link">
+    <visual>
+      <origin xyz="0 0 0" rpy="0 0 0"/>
+      <geometry>
+        <mesh
+          filename="package://boe_robot_description/meshes/caster_base_link.STL"/>
+      </geometry>
+      <material name="body_color"/>
+    </visual>
+  </link>
+  <joint name="caster_base_joint" type="fixed">
+    <parent link="base_link"/>
+    <child link="caster_base_link"/>
+    <origin
+      xyz="-0.0049954073 -0.0042939669 0.0185737626"
+      rpy="0 0 0"/>
+  </joint>
+  <!-- Phần caster có thể tự xoay theo hướng chuyển động -->
+  <link name="caster_rotation_link">
+    <visual>
+      <origin xyz="0 0 0" rpy="0 0 0"/>
+      <geometry>
+        <mesh
+          filename="package://boe_robot_description/meshes/caster_rotation_link.STL"/>
+      </geometry>
+      <material name="body_color"/>
+    </visual>
+  </link>
+  <joint name="caster_rotation_joint" type="continuous">
+    <parent link="caster_base_link"/>
+    <child link="caster_rotation_link"/>
+    <origin
+      xyz="-0.0361714130 0 -0.0106540966"
+      rpy="0 0 0"/>
+    <axis xyz="0 0 1"/>
+    <limit effort="0.5" velocity="10.0"/>
+  </joint>
+  <!-- Bánh caster có thể lăn tự do -->
+  <link name="caster_wheel_link">
+    <visual>
+      <origin xyz="0 0 0" rpy="0 0 0"/>
+      <geometry>
+        <mesh
+          filename="package://boe_robot_description/meshes/caster_wheel_link.STL"/>
+      </geometry>
+      <material name="wheel_color"/>
+    </visual>
+  </link>
+  <joint name="caster_wheel_joint" type="continuous">
+    <parent link="caster_rotation_link"/>
+    <child link="caster_wheel_link"/>
+    <origin
+      xyz="0.0179800159 0.0039088610 -0.023"
+      rpy="-1.5707963268 0 0"/>
+    <axis xyz="-0.0665291474 0 0.9977844820"/>
+    <limit effort="0.5" velocity="20.0"/>
+  </joint>
 </robot>

Commit message: them lidar

File: boe_robot_description/urdf/boe_robot.urdf.xacro (robot description, xacro)
@@ -144,3 +144,28 @@
     <limit effort="0.5" velocity="20.0"/>
   </joint>
+    <!-- ====================================================== -->
+  <!-- LiDAR 2D                                               -->
+  <!-- ====================================================== -->
+  <material name="lidar_color">
+    <color rgba="0.15 0.15 0.15 1.0"/>
+  </material>
+  <!-- Phần thân của cảm biến LiDAR -->
+  <link name="lidar_link">
+    <visual>
+      <origin xyz="0 0 0" rpy="0 0 0"/>
+      <geometry>
+        <mesh
+          filename="package://boe_robot_description/meshes/lidar_link.STL"/>
+      </geometry>
+      <material name="lidar_color"/>
+    </visual>
+  </link>
+  <!-- LiDAR được gắn cố định trên thân xe -->
+  <joint name="lidar_joint" type="fixed">
+    <parent link="base_link"/>
+    <child link="lidar_link"/>
+    <origin
+      xyz="-0.0070723108 -0.0045653019 0.0434219487"
+      rpy="0 0 0"/>
+  </joint>
 </robot>

Commit message: thêm thuộc tính vật lý cho base_link và 2 bánh chủ động

File: boe_robot_description/urdf/boe_robot.urdf.xacro (robot description, xacro)
@@ -5,4 +5,5 @@
   <!-- Các thông số chính của robot -->
   <xacro:property name="wheel_radius" value="0.03272"/>
+  <xacro:property name="wheel_width" value="0.00975"/>
   <xacro:property name="wheel_separation" value="0.115"/>
   <!-- Màu thân xe -->
@@ -32,6 +33,7 @@
       rpy="0 0 0"/>
   </joint>
-  <!-- Thân xe -->
+    <!-- Thân xe -->
   <link name="base_link">
+    <!-- Hình dạng hiển thị -->
     <visual>
       <origin xyz="0 0 0" rpy="0 0 0"/>
@@ -42,7 +44,31 @@
       <material name="body_color"/>
     </visual>
-  </link>
-  <!-- Bánh chủ động bên trái -->
+    <!-- Hình dạng dùng để tính va chạm -->
+    <collision>
+      <origin
+        xyz="-0.0018954 -0.0042940 0.0018238"
+        rpy="0 0 0"/>
+      <geometry>
+        <box size="0.1209 0.1150 0.0335"/>
+      </geometry>
+    </collision>
+    <!-- Khối lượng và mô-men quán tính -->
+    <inertial>
+      <origin
+        xyz="0.0154452 -0.0042940 0.0038704"
+        rpy="0 0 0"/>
+      <mass value="0.0814944"/>
+      <inertia
+        ixx="2.7770132e-05"
+        ixy="0.0"
+        ixz="1.0575890e-06"
+        iyy="4.2579467e-05"
+        iyz="0.0"
+        izz="6.3174700e-05"/>
+    </inertial>
+  </link>
+    <!-- Bánh chủ động bên trái -->
   <link name="wheel_left_link">
+    <!-- Hình dạng hiển thị -->
     <visual>
       <origin xyz="0 0 0" rpy="0 0 0"/>
@@ -53,4 +79,25 @@
       <material name="wheel_color"/>
     </visual>
+    <!-- Hình trụ dùng để tính tiếp xúc với mặt đất -->
+    <collision>
+      <origin xyz="0 0 -0.002125" rpy="0 0 0"/>
+      <geometry>
+        <cylinder
+          radius="${wheel_radius}"
+          length="${wheel_width}"/>
+      </geometry>
+    </collision>
+    <!-- Thông số vật lý bánh trái -->
+    <inertial>
+      <origin xyz="0 0 -0.0014620" rpy="0 0 0"/>
+      <mass value="0.0130643"/>
+      <inertia
+        ixx="4.3289310e-06"
+        ixy="0.0"
+        ixz="0.0"
+        iyy="4.3289308e-06"
+        iyz="0.0"
+        izz="8.5765717e-06"/>
+    </inertial>
   </link>
   <joint name="wheel_left_joint" type="continuous">
@@ -65,4 +112,5 @@
   <!-- Bánh chủ động bên phải -->
   <link name="wheel_right_link">
+    <!-- Hình dạng hiển thị -->
     <visual>
       <origin xyz="0 0 0" rpy="0 0 0"/>
@@ -73,4 +121,25 @@
       <material name="wheel_color"/>
     </visual>
+    <!-- Hình trụ dùng để tính tiếp xúc với mặt đất -->
+    <collision>
+      <origin xyz="0 0 -0.002125" rpy="0 0 0"/>
+      <geometry>
+        <cylinder
+          radius="${wheel_radius}"
+          length="${wheel_width}"/>
+      </geometry>
+    </collision>
+    <!-- Thông số vật lý bánh phải -->
+    <inertial>
+      <origin xyz="0 0 -0.0014620" rpy="0 0 0"/>
+      <mass value="0.0130643"/>
+      <inertia
+        ixx="4.3289310e-06"
+        ixy="0.0"
+        ixz="0.0"
+        iyy="4.3289308e-06"
+        iyz="0.0"
+        izz="8.5765717e-06"/>
+    </inertial>
   </link>
   <joint name="wheel_right_joint" type="continuous">

Commit message: 7. thêm collision và inertial cho caster và LiDAR

File: boe_robot_description/urdf/boe_robot.urdf.xacro (robot description, xacro)
@@ -7,4 +7,6 @@
   <xacro:property name="wheel_width" value="0.00975"/>
   <xacro:property name="wheel_separation" value="0.115"/>
+  <xacro:property name="caster_wheel_radius" value="0.01805"/>
+  <xacro:property name="caster_wheel_width" value="0.02135"/>
   <!-- Màu thân xe -->
   <material name="body_color">
@@ -165,4 +167,25 @@
       <material name="body_color"/>
     </visual>
+    <collision>
+      <origin
+        xyz="-0.0361715 0 -0.0059156"
+        rpy="0 0 0"/>
+      <geometry>
+        <box size="0.02925 0.04230 0.00883"/>
+      </geometry>
+    </collision>
+    <inertial>
+      <origin
+        xyz="-0.0361715 0 -0.0030658"
+        rpy="0 0 0"/>
+      <mass value="0.0030125"/>
+      <inertia
+        ixx="3.9104173e-07"
+        ixy="0.0"
+        ixz="0.0"
+        iyy="2.0299201e-07"
+        iyz="0.0"
+        izz="5.8856957e-07"/>
+    </inertial>
   </link>
   <joint name="caster_base_joint" type="fixed">
@@ -183,4 +206,25 @@
       <material name="body_color"/>
     </visual>
+    <collision>
+      <origin
+        xyz="0.0075675 0.0003090 -0.0147200"
+        rpy="0 0 0"/>
+      <geometry>
+        <box size="0.04273 0.02820 0.03036"/>
+      </geometry>
+    </collision>
+    <inertial>
+      <origin
+        xyz="0.0080981 0.0017545 -0.0072399"
+        rpy="0 0 0"/>
+      <mass value="0.0011340"/>
+      <inertia
+        ixx="1.7627566e-07"
+        ixy="-8.3344816e-09"
+        ixz="3.7574602e-08"
+        iyy="2.1288142e-07"
+        iyz="8.1503549e-09"
+        izz="2.2080115e-07"/>
+    </inertial>
   </link>
   <joint name="caster_rotation_joint" type="continuous">
@@ -191,4 +235,5 @@
       rpy="0 0 0"/>
     <axis xyz="0 0 1"/>
+    <dynamics damping="0.02" friction="0.0"/>
     <limit effort="0.5" velocity="10.0"/>
   </joint>
@@ -203,4 +248,25 @@
       <material name="wheel_color"/>
     </visual>
+    <collision>
+      <origin xyz="0 0 0" rpy="0 0 0"/>
+      <geometry>
+        <cylinder
+          radius="${caster_wheel_radius}"
+          length="${caster_wheel_width}"/>
+      </geometry>
+    </collision>
+    <inertial>
+      <origin
+        xyz="-0.0000022 0 0.0000102"
+        rpy="0 0 0"/>
+      <mass value="0.0076789"/>
+      <inertia
+        ixx="8.3385020e-07"
+        ixy="0.0"
+        ixz="-1.2263852e-07"
+        iyy="8.0727807e-07"
+        iyz="0.0"
+        izz="1.3732925e-06"/>
+    </inertial>
   </link>
   <joint name="caster_wheel_joint" type="continuous">
@@ -211,4 +277,5 @@
       rpy="-1.5707963268 0 0"/>
     <axis xyz="-0.0665291474 0 0.9977844820"/>
+    <dynamics damping="0.01" friction="0.0"/>
     <limit effort="0.5" velocity="20.0"/>
   </joint>
@@ -229,4 +296,25 @@
       <material name="lidar_color"/>
     </visual>
+    <collision>
+      <origin
+        xyz="0.0044570 0.0002393 -0.0043482"
+        rpy="0 0 0"/>
+      <geometry>
+        <cylinder radius="0.038" length="0.041"/>
+      </geometry>
+    </collision>
+    <inertial>
+      <origin
+        xyz="0.0038634 0.0002219 -0.0055496"
+        rpy="0 0 0"/>
+      <mass value="0.1653828"/>
+      <inertia
+        ixx="7.8845557e-05"
+        ixy="2.7219327e-07"
+        ixz="2.1789506e-06"
+        iyy="7.5209918e-05"
+        iyz="1.6227741e-07"
+        izz="1.0994675e-04"/>
+    </inertial>
   </link>
   <!-- LiDAR được gắn cố định trên thân xe -->

Commit message: 8. package Gazebo

File: boe_robot_description/urdf/boe_robot.urdf.xacro (robot description, xacro)
@@ -70,18 +70,19 @@
     </inertial>
   </link>
-    <!-- Bánh chủ động bên trái -->
+  <!-- Bánh chủ động bên trái -->
   <link name="wheel_left_link">
-    <!-- Hình dạng hiển thị -->
-    <visual>
-      <origin xyz="0 0 0" rpy="0 0 0"/>
-      <geometry>
-        <mesh
-          filename="package://boe_robot_description/meshes/wheel_left_link.STL"/>
+    <visual>
+      <origin
+        xyz="0 0 0"
+        rpy="1.5707963268 0 0"/>
+      <geometry>
+        <mesh filename="package://boe_robot_description/meshes/wheel_left_link.STL"/>
       </geometry>
       <material name="wheel_color"/>
     </visual>
-    <!-- Hình trụ dùng để tính tiếp xúc với mặt đất -->
-    <collision>
-      <origin xyz="0 0 -0.002125" rpy="0 0 0"/>
+    <collision>
+      <origin
+        xyz="0 0.002125 0"
+        rpy="1.5707963268 0 0"/>
       <geometry>
         <cylinder
@@ -90,7 +91,8 @@
       </geometry>
     </collision>
-    <!-- Thông số vật lý bánh trái -->
-    <inertial>
-      <origin xyz="0 0 -0.0014620" rpy="0 0 0"/>
+    <inertial>
+      <origin
+        xyz="0 0.0014620 0"
+        rpy="1.5707963268 0 0"/>
       <mass value="0.0130643"/>
       <inertia
@@ -108,22 +110,23 @@
     <origin
       xyz="0.0329316266 0.0532060331 0.0005737626"
-      rpy="1.5707963268 0 3.1415926536"/>
-    <axis xyz="0 0 1"/>
+      rpy="0 0 0"/>
+    <axis xyz="0 1 0"/>
     <limit effort="1.0" velocity="20.0"/>
   </joint>
   <!-- Bánh chủ động bên phải -->
   <link name="wheel_right_link">
-    <!-- Hình dạng hiển thị -->
-    <visual>
-      <origin xyz="0 0 0" rpy="0 0 0"/>
-      <geometry>
-        <mesh
-          filename="package://boe_robot_description/meshes/wheel_right_link.STL"/>
+    <visual>
+      <origin
+        xyz="0 0 0"
+        rpy="-1.5707963268 0 0"/>
+      <geometry>
+        <mesh filename="package://boe_robot_description/meshes/wheel_right_link.STL"/>
       </geometry>
       <material name="wheel_color"/>
     </visual>
-    <!-- Hình trụ dùng để tính tiếp xúc với mặt đất -->
-    <collision>
-      <origin xyz="0 0 -0.002125" rpy="0 0 0"/>
+    <collision>
+      <origin
+        xyz="0 -0.002125 0"
+        rpy="-1.5707963268 0 0"/>
       <geometry>
         <cylinder
@@ -132,7 +135,8 @@
       </geometry>
     </collision>
-    <!-- Thông số vật lý bánh phải -->
-    <inertial>
-      <origin xyz="0 0 -0.0014620" rpy="0 0 0"/>
+    <inertial>
+      <origin
+        xyz="0 -0.0014620 0"
+        rpy="-1.5707963268 0 0"/>
       <mass value="0.0130643"/>
       <inertia
@@ -150,6 +154,6 @@
     <origin
       xyz="0.0309316266 -0.0617939669 0.0005737626"
-      rpy="1.5707963268 0 0"/>
-    <axis xyz="0 0 -1"/>
+      rpy="0 0 0"/>
+    <axis xyz="0 1 0"/>
     <limit effort="1.0" velocity="20.0"/>
   </joint>
@@ -157,5 +161,5 @@
   <!-- Cụm bánh caster                                       -->
   <!-- ====================================================== -->
-  <!-- Đế caster được gắn cố định với thân robot -->
+  <!-- Đế caster gắn cố định với thân robot -->
   <link name="caster_base_link">
     <visual>
@@ -241,5 +245,7 @@
   <link name="caster_wheel_link">
     <visual>
-      <origin xyz="0 0 0" rpy="0 0 0"/>
+      <origin
+        xyz="0 0 0"
+        rpy="-1.5707963268 0 0"/>
       <geometry>
         <mesh
@@ -249,5 +255,7 @@
     </visual>
     <collision>
-      <origin xyz="0 0 0" rpy="0 0 0"/>
+      <origin
+        xyz="0 0 0"
+        rpy="-1.5707963268 0 0"/>
       <geometry>
         <cylinder
@@ -258,6 +266,6 @@
     <inertial>
       <origin
-        xyz="-0.0000022 0 0.0000102"
-        rpy="0 0 0"/>
+        xyz="-0.0000022 0.0000102 0"
+        rpy="-1.5707963268 0 0"/>
       <mass value="0.0076789"/>
       <inertia
@@ -275,10 +283,10 @@
     <origin
       xyz="0.0179800159 0.0039088610 -0.023"
-      rpy="-1.5707963268 0 0"/>
-    <axis xyz="-0.0665291474 0 0.9977844820"/>
+      rpy="0 0 0"/>
+    <axis xyz="0 1 0"/>
     <dynamics damping="0.01" friction="0.0"/>
     <limit effort="0.5" velocity="20.0"/>
   </joint>
-    <!-- ====================================================== -->
+  <!-- ====================================================== -->
   <!-- LiDAR 2D                                               -->
   <!-- ====================================================== -->

Commit message: vẫn là package gazebo

File: boe_robot_description/urdf/boe_robot.urdf.xacro (robot description, xacro)
@@ -232,4 +232,5 @@
     </inertial>
   </link>
+  <!-- Khớp thụ động cho cả cụm caster đổi hướng quanh trục Z. -->
   <joint name="caster_rotation_joint" type="continuous">
     <parent link="caster_base_link"/>
@@ -239,8 +240,8 @@
       rpy="0 0 0"/>
     <axis xyz="0 0 1"/>
-    <dynamics damping="0.02" friction="0.0"/>
-    <limit effort="0.5" velocity="10.0"/>
-  </joint>
-  <!-- Bánh caster có thể lăn tự do -->
+    <dynamics damping="0.02" friction="0.001"/>
+    <limit effort="0.2" velocity="10.0"/>
+  </joint>
+  <!-- Bánh caster hiển thị; collision vật lý đơn giản nằm trong SDF. -->
   <link name="caster_wheel_link">
     <visual>
@@ -278,13 +279,14 @@
     </inertial>
   </link>
+  <!-- Khớp thụ động cho bánh caster lăn quanh trục Y. -->
   <joint name="caster_wheel_joint" type="continuous">
     <parent link="caster_rotation_link"/>
     <child link="caster_wheel_link"/>
     <origin
-      xyz="0.0179800159 0.0039088610 -0.023"
+      xyz="0.0179800159 0.0039088610 -0.0220196660"
       rpy="0 0 0"/>
     <axis xyz="0 1 0"/>
-    <dynamics damping="0.01" friction="0.0"/>
-    <limit effort="0.5" velocity="20.0"/>
+    <dynamics damping="0.005" friction="0.001"/>
+    <limit effort="0.2" velocity="20.0"/>
   </joint>
   <!-- ====================================================== -->
